File: OPMBoard.kicad_sch (KiCad schematic)
At the start: 48 parts, among them J1 USB_C_Receptacle_USB2.0, J2 Conn_01x03, J3 Conn_02x10_Counter_Clockwise, J4 AudioJack3, SW1 SW_SPDT, U1 NJM4580, U2 NJM4580, U3 NJM4580, U4 YM2151, U5 YM3012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

Commit message: Update schematic
Parts:
- removed J3: Conn_02x10_Counter_Clockwise, Connector_PinHeader_2.54mm:PinHeader_2x10_P2.54mm_Vertical, symbol Connector_Generic:Conn_02x10_Counter_Clockwise
- removed PS1: ITQ2415S, Converter_DCDC:Converter_DCDC_XP_POWER-ITxxxxxS_THT, symbol Converter_DCDC:ITQ2415S
- added FID1: Fiducial, Fiducial:Fiducial_0.5mm_Mask1mm, symbol Mechanical:Fiducial
- added H1, H2, H3, H4: MountingHole, MountingHole:MountingHole_3.2mm_M3, symbol Mechanical:MountingHole
- added J2: Conn_02x12_Odd_Even, Connector_PinHeader_2.54mm:PinHeader_2x12_P2.54mm_Vertical, symbol Connector_Generic:Conn_02x12_Odd_Even
- added PS1: ITX0505S-R, Converter_DCDC:Converter_DCDC_XP_POWER-ITxxxxxS_THT, symbol Converter_DCDC:ITX0505S-R
- added RN1: 4.7k * 8, Resistor_THT:R_Array_SIP9, symbol Device:R_Network08
- C10, C11: footprint Capacitor_THT:CP_Radial_D10.0mm_P7.50mm -> Capacitor_THT:CP_Radial_D5.0mm_P2.00mm
- C8, C9: footprint Capacitor_THT:CP_Radial_D10.0mm_P7.50mm -> Capacitor_THT:CP_Radial_D5.0mm_P2.50mm
- D1: value 12V_GREEN -> 5V_GREEN
- D2: value 5V_GREEN -> VDD_GREEN
- D3: value -12V_GREEN -> -5V_GREEN
- R1: value 100 -> 270
- R2, R4: value 9.1k -> 2k
- X1: footprint Oscillator:Oscillator_DIP-14_LargePads -> MayLib:Oscillator_DIP-14_Full
- X2: footprint Oscillator:Oscillator_DIP-8_LargePads -> MayLib:Oscillator_DIP-8_Full
- renumbered J2 to J3
Connections:
- net +12V is gone; now on net +5V: C1.1, J3.1 (Pin_1), R2.1, R5.1, U1.8 (V+), U2.8 (V+), U3.8 (V+)
- net +5V: now also J2.1 (Pin_1), J2.2 (Pin_2), PS1.6 (+Vout), RN1.1 (common); no longer C6.1, C7.1, L1.2, R3.1, U4.22 (VDD), U5.1 (VDD)
- net A0: now also J2.21 (Pin_21)
- net CT1: now also J2.17 (Pin_17)
- net CT2: now also J2.19 (Pin_19)
- net D0: now also J2.6 (Pin_6)
- net D1: now also J2.8 (Pin_8)
- net D2: now also J2.10 (Pin_10)
- net D3: now also J2.12 (Pin_12)
- net D4: now also J2.14 (Pin_14)
- net D5: now also J2.16 (Pin_16)
- net D6: now also J2.18 (Pin_18)
- net D7: now also J2.20 (Pin_20)
- net GND: now also U5.16 (AGND), U5.8 (AGND), J2.22 (Pin_22), J2.23 (Pin_23), J2.24 (Pin_24), J2.3 (Pin_3), J2.4 (Pin_4), PS1.1 (-Vin), PS1.3 (OnOff)
- net GNDA: now also PS1.7 (Common); no longer U5.16 (AGND), U5.8 (AGND)
- net ~{CS}: now also J2.15 (Pin_15), RN1.9 (R8)
- net ~{ICL}: now also J2.9 (Pin_9), RN1.4 (R3)
- net ~{IC}: now also J2.7 (Pin_7), RN1.6 (R5)
- net ~{IRQ}: now also J2.5 (Pin_5), RN1.5 (R4)
- net ~{RD}: now also J2.13 (Pin_13), RN1.8 (R7)
- net ~{WR}: now also J2.11 (Pin_11), RN1.7 (R6)
- net -12V renamed -5V
- net -5V: now also PS1.8 (-Vout)
- new net VDD: C6.1, C7.1, L1.2, PS1.2 (+Vin), R3.1, U4.22 (VDD), U5.1 (VDD)
- no-connect marks 9 -> 11
Other:
- moved on the sheet: C5, C6, J3, J4, JP2, L1, U2C
